File: hardware/coupon/coupon.kicad_sch (KiCad schematic)
At the start: 80 parts, among them SW1 tactile

Commit message: hw(coupon): the pot is Alpha by measurement, and the bulk caps get their volts
Three of the five order blockers close at the desk. The Alps RK09K
footprint is disproven pad for pad against KiCad's own library: pins
1/2/3 match the Alpha exactly (2.5 mm in-line), the support lugs do not
(0.5 mm out, 0.4 mm down), so the coupon now carries the Alpha
RD901F-40 vertical footprint -- the part the note always named, and the
one Electrosmith's example uses. Linear 20 k in 9 mm vertical is a real
Alpha part (B20K), stocked by Tayda, Thonk and Exploding Shed. The four
10u bulk caps become '10u 25V' X5R as one BOM line item; the 12 V pair
needs the rating and the 3V3 pair rides along.

Proof chain re-run: netlist matches node for node, zero collisions, ERC
still the three explained violations. Still open before the order: the
bus board measurement and the Patch SM land-pattern risk.

Co-Authored-By: HAL 9000 <293417720+bea-ton-k@users.noreply.github.com>
Parts:
- C_B3V3, C_BA3V3, C_BN12, C_BP12: value 10u -> 10u 25V
- RV1, RV2, RV3, RV4, RV5, RV6, RV7: footprint Potentiometer_THT:Potentiometer_Alps_RK09K_Single_Vertical -> Potentiometer_THT:Potentiometer_Alpha_RD901F-40-00D_Single_Vertical

Commit message: hw(coupon): four 2x5 sockets, vertical pots, and the first powered board
The Patch SM landing pattern is four separate 2x5 groups, not two 2x10
rows, so the socket BOM lines become J_SM1..J_SM4, each cut from one of
the four 2x10 strips already bought. The stock right-angle pots turned
out to reach the board only on flying leads, which the coupon may not be
built with; order-bom.md now names an RV09 vertical part as the one open
order line and records that Reichelt carries no 20k in that size.

The README gains the bring-up record of 2026-09-17: the unpowered meter
signatures that identify the ground pads and bank A without counting,
the 1.6 kOhm reading that proves both jumpers conduct, and the moat
continuity check that can no longer be taken on this board.

Regenerated and checked on 2026-09-27: build.py reproduces the schematic
up to its unseeded UUIDs, review.py and assembly_plan.py reproduce their
outputs byte for byte.

Co-Authored-By: HAL 9000 <293417720+bea-ton-k@users.noreply.github.com>
Parts:
- removed J_SM1, J_SM2: 2x10 socket 2.54mm, symbol Connector_Generic:Conn_02x10_Odd_Even
- added J_SM1, J_SM2, J_SM3, J_SM4: 2x5 socket 2.54mm, symbol Connector_Generic:Conn_02x05_Odd_Even
