File: hardware/reva/kicad/power.kicad_sch (KiCad schematic)
At the start: 10 parts

Commit message: hw(reva): SD socket decoupling and a DNP tantalum option at the AMS1117
Co-Authored-By: HAL 9000 <293417720+bea-ton-k@users.noreply.github.com>
Parts:
- added C_LDO_T: 22u 16V tant, Capacitor_Tantalum_SMD:CP_EIA-6032-28_Kemet-C, symbol Device:C_Polarized
Connections:
- net 3V3D: now also C_LDO_T.1
- net GND: now also C_LDO_T.2
Changed lines of the file:
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@@
 	)
 	(symbol
-		(lib_id "power:PWR_FLAG")
-		(at 312.42 25.4 0)
+		(lib_id "Device:C_Polarized")
+		(at 312.42 39.37 0)
 		(unit 1)
 		(exclude_from_sim no)
-		(in_bom no)
-		(on_board no)
-		(dnp no)
-		(property "Reference" "#FLG0001"
-			(at 312.42 20.32 0)
-			(effects (font (size 1.27 1.27)) (justify left) (hide yes)))
-		(property "Value" "PWR_FLAG"
-			(at 312.42 22.86 0)
-			(effects (font (size 1.27 1.27)) (justify left) (hide yes)))
-		(property "Footprint" ""
-			(at 312.42 25.4 0)
+		(in_bom yes)
+		(on_board yes)
+		(dnp yes)
+		(property "Reference" "C_LDO_T"
+			(at 312.42 19.05 0)
+			(effects (font (size 1.27 1.27)) (justify left)))
+		(property "Value" "22u 16V tant"
+			(at 312.42 21.59 0)
+			(effects (font (size 1.27 1.27)) (justify left)))
+		(property "Footprint" "Capacitor_Tantalum_SMD:CP_EIA-6032-28_Kemet-C"
+			(at 312.42 39.37 0)
 			(effects (font (size 1.27 1.27)) (justify left) (hide yes)))
 		(property "Datasheet" ""
-			(at 312.42 25.4 0)
+			(at 312.42 39.37 0)
 			(effects (font (size 1.27 1.27)) (justify left) (hide yes)))
-		(property "Description" ""
-			(at 312.42 25.4 0)
+		(property "Description" "DNP bring-up option: fit if the regulator oscillates with the MLCC alone"
+			(at 312.42 39.37 0)
+			(effects (font (size 1.27 1.27)) (justify left) (hide yes)))
+		(property "LCSC" "C1967941"
+			(at 312.42 39.37 0)
 			(effects (font (size 1.27 1.27)) (justify left) (hide yes)))
 		(pin "1")
+		(pin "2")
 		(instances
 			(project "reva"
-				(path "/f95ef33a-cefb-5011-a30f-e0d40d3b300b/565f096c-3c93-5bb3-ae29-71358df00935" (reference "#FLG0001") (unit 1))))
+				(path "/f95ef33a-cefb-5011-a30f-e0d40d3b300b/565f096c-3c93-5bb3-ae29-71358df00935" (reference "C_LDO_T") (unit 1))))
 	)
-	(wire (pts (xy 312.42 25.4) (xy 312.42 29.21))
+	(wire (pts (xy 312.42 43.18) (xy 312.42 46.99))
 		(stroke (width 0) (type default)))
 	(symbol
-		(lib_id "power:+12V")
-		(at 312.42 29.21 180)
+		(lib_id "power:GND")
+		(at 312.42 46.99 0)
 		(unit 1)
 		(exclude_from_sim no)
@@
 		(dnp no)
 		(property "Reference" "#PWR0020"
-			(at 312.42 29.21 0)
+			(at 312.42 46.99 0)
 			(effects (font (size 1.27 1.27)) (justify left) (hide yes)))
-		(property "Value" "+12V"
-			(at 312.42 34.29 0)
+		(property "Value" "GND"
+			(at 312.42 52.07 0)
 			(effects (font (size 1.27 1.27))))
 		(property "Footprint" ""
-			(at 312.42 29.21 0)
+			(at 312.42 46.99 0)
 			(effects (font (size 1.27 1.27)) (justify left) (hide yes)))
 		(property "Datasheet" ""
-			(at 312.42 29.21 0)
+			(at 312.42 46.99 0)
 			(effects (font (size 1.27 1.27)) (justify left) (hide yes)))
 		(pin "1")
@@
 			(project "reva"
 				(path "/f95ef33a-cefb-5011-a30f-e0d40d3b300b/565f096c-3c93-5bb3-ae29-71358df00935" (reference "#PWR0020") (unit 1))))
+	)
+	(wire (pts (xy 312.42 35.56) (xy 312.42 31.75))
+		(stroke (width 0) (type default)))
+	(symbol
+		(lib_id "power:+3V3")
+		(at 312.42 31.75 0)
+		(unit 1)
+		(exclude_from_sim no)
+		(in_bom no)
+		(on_board no)
+		(dnp no)
+		(property "Reference" "#PWR0021"
+			(at 312.42 31.75 0)
+			(effects (font (size 1.27 1.27)) (justify left) (hide yes)))
+		(property "Value" "3V3D"
+			(at 312.42 26.67 0)
+			(effects (font (size 1.27 1.27))))
+		(property "Footprint" ""
+			(at 312.42 31.75 0)
+			(effects (font (size 1.27 1.27)) (justify left) (hide yes)))
+		(property "Datasheet" ""
+			(at 312.42 31.75 0)
+			(effects (font (size 1.27 1.27)) (justify left) (hide yes)))
+		(pin "1")
+		(instances
+			(project "reva"
+				(path "/f95ef33a-cefb-5011-a30f-e0d40d3b300b/565f096c-3c93-5bb3-ae29-71358df00935" (reference "#PWR0021") (unit 1))))
 	)
 	(symbol
@@
 		(on_board no)
 		(dnp no)
-		(property "Reference" "#FLG0002"
+		(property "Reference" "#FLG0001"
 			(at 328.93 20.32 0)
 			(effects (font (size 1.27 1.27)) (justify left) (hide yes)))
@@
 		(instances
 			(project "reva"
-				(path "/f95ef33a-cefb-5011-a30f-e0d40d3b300b/565f096c-3c93-5bb3-ae29-71358df00935" (reference "#FLG0002") (unit 1))))
+				(path "/f95ef33a-cefb-5011-a30f-e0d40d3b300b/565f096c-3c93-5bb3-ae29-71358df00935" (reference "#FLG0001") (unit 1))))
 	)
 	(wire (pts (xy 328.93 25.4) (xy 328.93 29.21))
 		(stroke (width 0) (type default)))
 	(symbol
-		(lib_id "power:-12V")
+		(lib_id "power:+12V")
 		(at 328.93 29.21 180)
 		(unit 1)
@@
 		(on_board no)
 		(dnp no)
-		(property "Reference" "#PWR0021"
+		(property "Reference" "#PWR0022"
 			(at 328.93 29.21 0)
 			(effects (font (size 1.27 1.27)) (justify left) (hide yes)))
-		(property "Value" "-12V"
+		(property "Value" "+12V"
 			(at 328.93 34.29 0)
 			(effects (font (size 1.27 1.27))))
@@
 		(instances
 			(project "reva"
-				(path "/f95ef33a-cefb-5011-a30f-e0d40d3b300b/565f096c-3c93-5bb3-ae29-71358df00935" (reference "#PWR0021") (unit 1))))
+				(path "/f95ef33a-cefb-5011-a30f-e0d40d3b300b/565f096c-3c93-5bb3-ae29-71358df00935" (reference "#PWR0022") (unit 1))))
+	)
+	(symbol
+		(lib_id "power:PWR_FLAG")
+		(at 344.17 25.4 0)
+		(unit 1)
+		(exclude_from_sim no)
+		(in_bom no)
+		(on_board no)
+		(dnp no)
+		(property "Reference" "#FLG0002"
+			(at 344.17 20.32 0)
+			(effects (font (size 1.27 1.27)) (justify left) (hide yes)))
+		(property "Value" "PWR_FLAG"
+			(at 344.17 22.86 0)
+			(effects (font (size 1.27 1.27)) (justify left) (hide yes)))
+		(property "Footprint" ""
+			(at 344.17 25.4 0)
+			(effects (font (size 1.27 1.27)) (justify left) (hide yes)))
+		(property "Datasheet" ""
+			(at 344.17 25.4 0)
+			(effects (font (size 1.27 1.27)) (justify left) (hide yes)))
+		(property "Description" ""
+			(at 344.17 25.4 0)
+			(effects (font (size 1.27 1.27)) (justify left) (hide yes)))
+		(pin "1")
+		(instances
+			(project "reva"
+				(path "/f95ef33a-cefb-5011-a30f-e0d40d3b300b/565f096c-3c93-5bb3-ae29-71358df00935" (reference "#FLG0002") (unit 1))))
+	)
+	(wire (pts (xy 344.17 25.4) (xy 344.17 29.21))
+		(stroke (width 0) (type default)))
+	(symbol
+		(lib_id "power:-12V")
+		(at 344.17 29.21 180)
+		(unit 1)
+		(exclude_from_sim no)
+		(in_bom no)
+		(on_board no)
+		(dnp no)
+		(property "Reference" "#PWR0023"
+			(at 344.17 29.21 0)
+			(effects (font (size 1.27 1.27)) (justify left) (hide yes)))
+		(property "Value" "-12V"
+			(at 344.17 34.29 0)
+			(effects (font (size 1.27 1.27))))
+		(property "Footprint" ""
+			(at 344.17 29.21 0)
+			(effects (font (size 1.27 1.27)) (justify left) (hide yes)))
+		(property "Datasheet" ""
+			(at 344.17 29.21 0)
+			(effects (font (size 1.27 1.27)) (justify left) (hide yes)))
+		(pin "1")
+		(instances
+			(project "reva"
+				(path "/f95ef33a-cefb-5011-a30f-e0d40d3b300b/565f096c-3c93-5bb3-ae29-71358df00935" (reference "#PWR0023") (unit 1))))
 	)
 	(embedded_fonts no)
