File: hardware/reva/kicad/sd.kicad_sch (KiCad schematic)
At the start: 1 part

Commit message: hw(reva): SD socket decoupling and a DNP tantalum option at the AMS1117
Co-Authored-By: HAL 9000 <293417720+bea-ton-k@users.noreply.github.com>
Parts:
- added C_SD1: 100n, Capacitor_SMD:C_0603_1608Metric, symbol Device:C
- added C_SD2: 10u 25V, Capacitor_SMD:C_0805_2012Metric, symbol Device:C
Connections:
- net GND: now also C_SD1.2, C_SD2.2
- net SM_3V3: now also C_SD1.1, C_SD2.1
Changed lines of the file:
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@@
 		(on_board no)
 		(dnp no)
-		(property "Reference" "#PWR0304"
+		(property "Reference" "#PWR0306"
 			(at 30.48 39.37 0)
 			(effects (font (size 1.27 1.27)) (justify left) (hide yes)))
@@
 		(instances
 			(project "reva"
-				(path "/f95ef33a-cefb-5011-a30f-e0d40d3b300b/6d2ba21e-e015-5890-8566-f6f5893db8a2" (reference "#PWR0304") (unit 1))))
+				(path "/f95ef33a-cefb-5011-a30f-e0d40d3b300b/6d2ba21e-e015-5890-8566-f6f5893db8a2" (reference "#PWR0306") (unit 1))))
 	)
 	(wire (pts (xy 34.29 36.83) (xy 30.48 36.83))
@@
 		(on_board no)
 		(dnp no)
-		(property "Reference" "#PWR0305"
+		(property "Reference" "#PWR0307"
 			(at 30.48 34.29 0)
 			(effects (font (size 1.27 1.27)) (justify left) (hide yes)))
@@
 		(instances
 			(project "reva"
-				(path "/f95ef33a-cefb-5011-a30f-e0d40d3b300b/6d2ba21e-e015-5890-8566-f6f5893db8a2" (reference "#PWR0305") (unit 1))))
+				(path "/f95ef33a-cefb-5011-a30f-e0d40d3b300b/6d2ba21e-e015-5890-8566-f6f5893db8a2" (reference "#PWR0307") (unit 1))))
 	)
 	(wire (pts (xy 34.29 31.75) (xy 30.48 31.75))
@@
 		(on_board no)
 		(dnp no)
-		(property "Reference" "#PWR0306"
+		(property "Reference" "#PWR0308"
 			(at 81.28 49.53 0)
 			(effects (font (size 1.27 1.27)) (justify left) (hide yes)))
@@
 		(instances
 			(project "reva"
-				(path "/f95ef33a-cefb-5011-a30f-e0d40d3b300b/6d2ba21e-e015-5890-8566-f6f5893db8a2" (reference "#PWR0306") (unit 1))))
+				(path "/f95ef33a-cefb-5011-a30f-e0d40d3b300b/6d2ba21e-e015-5890-8566-f6f5893db8a2" (reference "#PWR0308") (unit 1))))
+	)
+	(symbol
+		(lib_id "Device:C")
+		(at 104.14 39.37 0)
+		(unit 1)
+		(exclude_from_sim no)
+		(in_bom yes)
+		(on_board yes)
+		(dnp no)
+		(property "Reference" "C_SD1"
+			(at 104.14 19.05 0)
+			(effects (font (size 1.27 1.27)) (justify left)))
+		(property "Value" "100n"
+			(at 104.14 21.59 0)
+			(effects (font (size 1.27 1.27)) (justify left)))
+		(property "Footprint" "Capacitor_SMD:C_0603_1608Metric"
+			(at 104.14 39.37 0)
+			(effects (font (size 1.27 1.27)) (justify left) (hide yes)))
+		(property "Datasheet" ""
+			(at 104.14 39.37 0)
+			(effects (font (size 1.27 1.27)) (justify left) (hide yes)))
+		(property "Description" "SD socket VDD decoupling, at the socket"
+			(at 104.14 39.37 0)
+			(effects (font (size 1.27 1.27)) (justify left) (hide yes)))
+		(property "LCSC" "C14663"
+			(at 104.14 39.37 0)
+			(effects (font (size 1.27 1.27)) (justify left) (hide yes)))
+		(pin "1")
+		(pin "2")
+		(instances
+			(project "reva"
+				(path "/f95ef33a-cefb-5011-a30f-e0d40d3b300b/6d2ba21e-e015-5890-8566-f6f5893db8a2" (reference "C_SD1") (unit 1))))
+	)
+	(wire (pts (xy 104.14 43.18) (xy 104.14 46.99))
+		(stroke (width 0) (type default)))
+	(symbol
+		(lib_id "power:GND")
+		(at 104.14 46.99 0)
+		(unit 1)
+		(exclude_from_sim no)
+		(in_bom no)
+		(on_board no)
+		(dnp no)
+		(property "Reference" "#PWR0309"
+			(at 104.14 46.99 0)
+			(effects (font (size 1.27 1.27)) (justify left) (hide yes)))
+		(property "Value" "GND"
+			(at 104.14 52.07 0)
+			(effects (font (size 1.27 1.27))))
+		(property "Footprint" ""
+			(at 104.14 46.99 0)
+			(effects (font (size 1.27 1.27)) (justify left) (hide yes)))
+		(property "Datasheet" ""
+			(at 104.14 46.99 0)
+			(effects (font (size 1.27 1.27)) (justify left) (hide yes)))
+		(pin "1")
+		(instances
+			(project "reva"
+				(path "/f95ef33a-cefb-5011-a30f-e0d40d3b300b/6d2ba21e-e015-5890-8566-f6f5893db8a2" (reference "#PWR0309") (unit 1))))
+	)
+	(wire (pts (xy 104.14 35.56) (xy 104.14 31.75))
+		(stroke (width 0) (type default)))
+	(symbol
+		(lib_id "power:+3V3")
+		(at 104.14 31.75 0)
+		(unit 1)
+		(exclude_from_sim no)
+		(in_bom no)
+		(on_board no)
+		(dnp no)
+		(property "Reference" "#PWR0310"
+			(at 104.14 31.75 0)
+			(effects (font (size 1.27 1.27)) (justify left) (hide yes)))
+		(property "Value" "SM_3V3"
+			(at 104.14 26.67 0)
+			(effects (font (size 1.27 1.27))))
+		(property "Footprint" ""
+			(at 104.14 31.75 0)
+			(effects (font (size 1.27 1.27)) (justify left) (hide yes)))
+		(property "Datasheet" ""
+			(at 104.14 31.75 0)
+			(effects (font (size 1.27 1.27)) (justify left) (hide yes)))
+		(pin "1")
+		(instances
+			(project "reva"
+				(path "/f95ef33a-cefb-5011-a30f-e0d40d3b300b/6d2ba21e-e015-5890-8566-f6f5893db8a2" (reference "#PWR0310") (unit 1))))
+	)
+	(symbol
+		(lib_id "Device:C")
+		(at 121.92 39.37 0)
+		(unit 1)
+		(exclude_from_sim no)
+		(in_bom yes)
+		(on_board yes)
+		(dnp yes)
+		(property "Reference" "C_SD2"
+			(at 121.92 19.05 0)
+			(effects (font (size 1.27 1.27)) (justify left)))
+		(property "Value" "10u 25V"
+			(at 121.92 21.59 0)
+			(effects (font (size 1.27 1.27)) (justify left)))
+		(property "Footprint" "Capacitor_SMD:C_0805_2012Metric"
+			(at 121.92 39.37 0)
+			(effects (font (size 1.27 1.27)) (justify left) (hide yes)))
+		(property "Datasheet" ""
+			(at 121.92 39.37 0)
+			(effects (font (size 1.27 1.27)) (justify left) (hide yes)))
+		(property "Description" "DNP bring-up option: fit if the pot scan shows SD card noise"
+			(at 121.92 39.37 0)
+			(effects (font (size 1.27 1.27)) (justify left) (hide yes)))
+		(property "LCSC" "C15850"
+			(at 121.92 39.37 0)
+			(effects (font (size 1.27 1.27)) (justify left) (hide yes)))
+		(pin "1")
+		(pin "2")
+		(instances
+			(project "reva"
+				(path "/f95ef33a-cefb-5011-a30f-e0d40d3b300b/6d2ba21e-e015-5890-8566-f6f5893db8a2" (reference "C_SD2") (unit 1))))
+	)
+	(wire (pts (xy 121.92 43.18) (xy 121.92 46.99))
+		(stroke (width 0) (type default)))
+	(symbol
+		(lib_id "power:GND")
+		(at 121.92 46.99 0)
+		(unit 1)
+		(exclude_from_sim no)
+		(in_bom no)
+		(on_board no)
+		(dnp no)
+		(property "Reference" "#PWR0311"
+			(at 121.92 46.99 0)
+			(effects (font (size 1.27 1.27)) (justify left) (hide yes)))
+		(property "Value" "GND"
+			(at 121.92 52.07 0)
+			(effects (font (size 1.27 1.27))))
+		(property "Footprint" ""
+			(at 121.92 46.99 0)
+			(effects (font (size 1.27 1.27)) (justify left) (hide yes)))
+		(property "Datasheet" ""
+			(at 121.92 46.99 0)
+			(effects (font (size 1.27 1.27)) (justify left) (hide yes)))
+		(pin "1")
+		(instances
+			(project "reva"
+				(path "/f95ef33a-cefb-5011-a30f-e0d40d3b300b/6d2ba21e-e015-5890-8566-f6f5893db8a2" (reference "#PWR0311") (unit 1))))
+	)
+	(wire (pts (xy 121.92 35.56) (xy 121.92 31.75))
+		(stroke (width 0) (type default)))
+	(symbol
+		(lib_id "power:+3V3")
+		(at 121.92 31.75 0)
+		(unit 1)
+		(exclude_from_sim no)
+		(in_bom no)
+		(on_board no)
+		(dnp no)
+		(property "Reference" "#PWR0312"
+			(at 121.92 31.75 0)
+			(effects (font (size 1.27 1.27)) (justify left) (hide yes)))
+		(property "Value" "SM_3V3"
+			(at 121.92 26.67 0)
+			(effects (font (size 1.27 1.27))))
+		(property "Footprint" ""
+			(at 121.92 31.75 0)
+			(effects (font (size 1.27 1.27)) (justify left) (hide yes)))
+		(property "Datasheet" ""
+			(at 121.92 31.75 0)
+			(effects (font (size 1.27 1.27)) (justify left) (hide yes)))
+		(pin "1")
+		(instances
+			(project "reva"
+				(path "/f95ef33a-cefb-5011-a30f-e0d40d3b300b/6d2ba21e-e015-5890-8566-f6f5893db8a2" (reference "#PWR0312") (unit 1))))
 	)
 	(embedded_fonts no)

Commit message: hw(reva): J_SD is the Yamaichi PJS008U, footprint generated from LCSC's data
Co-Authored-By: HAL 9000 <293417720+bea-ton-k@users.noreply.github.com>
Parts:
- J_SD: footprint P4 -> FireFlow:SD_Yamaichi_PJS008U-3000-0; Source P4 -> hand-soldered
Changed lines of the file:
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@@
 			(at 57.15 22.86 0)
 			(effects (font (size 1.27 1.27)) (justify left)))
-		(property "Footprint" "P4"
+		(property "Footprint" "FireFlow:SD_Yamaichi_PJS008U-3000-0"
 			(at 57.15 34.29 0)
 			(effects (font (size 1.27 1.27)) (justify left) (hide yes)))
@@
 			(at 57.15 34.29 0)
 			(effects (font (size 1.27 1.27)) (justify left) (hide yes)))
-		(property "Description" "socket chosen in P4 (spec §6)"
+		(property "Description" "Yamaichi PJS008U-3000-0 vertical microSD, THT (P4-1 spec §4.2)"
 			(at 57.15 34.29 0)
 			(effects (font (size 1.27 1.27)) (justify left) (hide yes)))
-		(property "Source" "P4"
+		(property "Source" "hand-soldered"
 			(at 57.15 34.29 0)
 			(effects (font (size 1.27 1.27)) (justify left) (hide yes)))
