File: hardware/reva/kicad/reva.kicad_pcb (KiCad board)
At the start: 4 copper layers, 300.8 x 110 mm, 213 parts, among them J1 IN_L, J10 RESET, J11 MOD4_B, J12 MOD3_B, J13 MOD2_B, J14 MOD1_B, J15 GATE_B, J16 PITCH_B, J17 OUT_L, J18 OUT_R, J2 IN_R, J3 PITCH_A, J4 GATE_A, J5 MOD1_A, J6 MOD2_A, J7 MOD3_A, J8 MOD4_A, J9 CLOCK, SW1 REC_A, SW2 REC_B, SW3 MODBTN, SW4 SHIFTBTN

Commit message: hw(reva): spread the dense field west of the module through OVERRIDES (P4-2 convergence)
Nine OVERRIDES move U_SR2, U_SR3 west, U_IN1 and U_SR5 east of U_SM,
turn U_SR1 to rot 0 with R1-R3 in the pocket west of it, and put R12
next to U_MUX8. Field x 104-152, y 29-75: 146 -> 101 pads.
route.py (Task 6a run 2): 0 conflicts after 21 rounds, 284.9 s, 0 failed.

Co-Authored-By: HAL 9000 <293417720+bea-ton-k@users.noreply.github.com>
Parts:
- moved TP8 71.8 mm to (235.5, 68.2)
- moved C21 70.1 mm to (232.5, 71.0)
- moved U_SR5 59.8 mm to (230.0, 65.0), turned to 0 degrees
- moved TP9 59.5 mm to (227.5, 71.9)
- moved TP10 53.8 mm to (224.5, 68.2)
- moved TP15 50.8 mm to (230.5, 58.3)
- moved TP11 50.6 mm to (224.5, 65.4)
- moved TP12 47.9 mm to (224.5, 62.6)
- moved TP14 45.7 mm to (227.5, 58.1)
- moved TP13 44.8 mm to (224.5, 59.9)
- moved C22 44.6 mm to (197.3, 54.3)
- moved U_IN1 44.6 mm to (191.2, 56.8)
- moved TP5 43.0 mm to (150.9, 42.8)
- moved R12 33.6 mm to (170.0, 37.0), turned to 0 degrees
- moved R16 22.3 mm to (240.1, 82.8)
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
Commit message: hw(reva): keep plane-net pads clear of pot bodies; re-converge the router (P4-2)
U_SR3 moves to (84, 73) rot 90 and U_IN1 8 mm south, so U_SR3's GND pin,
C19 and C22 sit outside every pot body: no long stitch escape stub,
C19.2 stitched. U_SR5's offset is re-derived (its anchor follows them).
route.py: 0 conflicts after 22 rounds, 204.7 s, 0 failed; stitch
unresolved empty; every route_check step GREEN.

Co-Authored-By: HAL 9000 <293417720+bea-ton-k@users.noreply.github.com>
Parts:
- moved U_SR3 34.2 mm to (84.0, 73.0), turned to 90 degrees
- moved C19 25.0 mm to (90.0, 70.5), turned to 90 degrees
- moved U_REG 22.5 mm to (61.6, 55.0)
- moved C6 22.0 mm to (62.1, 71.0)
- moved D_N12 20.7 mm to (67.1, 74.5)
- moved C3 18.0 mm to (76.1, 70.5)
- moved C2 13.2 mm to (72.6, 70.0)
- moved C_LDO_T 11.0 mm to (72.6, 54.0)
- moved C5 10.5 mm to (72.6, 72.0), turned to 0 degrees
- moved C22 8.00 mm to (197.3, 62.3)
- moved U_IN1 8.00 mm to (191.2, 64.8)
- moved D_P12 7.52 mm to (74.6, 75.0)
- moved R14 6.00 mm to (143.9, 37.0)
- moved R15 4.00 mm to (196.0, 37.0)
- moved R16 4.00 mm to (240.1, 86.8)
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
Commit message: hw(reva): P4-2 the routed board committed, reva_route_guard
route.py owns hardware/reva/kicad/reva.kicad_pcb now; place.py --write
copies its renders only. reva_route_guard: two runs byte-identical, the
committed board fresh, every gated step green at baseline and red under
its own sabotage on its own lines, the KNOWN_PANEL name rule (spec 4.4),
zones apart, jack-zone members pinned, and branch probes for the
non-vacuity and count branches no sabotage reached. The drc sabotage
picks a decoupler whose loop keeps clear of foreign copper (C10's ran
into an M6_CH1 via; kicad-cli's report then varied run to run).

Co-Authored-By: HAL 9000 <293417720+bea-ton-k@users.noreply.github.com>
Routing:
- net MUX_S0: track 0.00 -> 516.6 mm, vias 0 -> 20
- net SR_CLK: track 0.00 -> 509.0 mm, vias 0 -> 31
- net MUX_S1: track 0.00 -> 508.6 mm, vias 0 -> 26
- net MUX_S2: track 0.00 -> 480.1 mm, vias 0 -> 21
- net 3V3D: track 0.00 -> 424.0 mm, vias 0 -> 31
- net SENSE_1: track 0.00 -> 263.6 mm, vias 0 -> 12
- net SR_LATCH: track 0.00 -> 226.3 mm, vias 0 -> 17
- net M6_CH3: track 0.00 -> 224.9 mm, vias 0 -> 12
- net KEY_SHIFTBTN: track 0.00 -> 209.9 mm, vias 0 -> 9
- net KEY_REC_A: track 0.00 -> 200.6 mm, vias 0 -> 10
- net SR_CHAIN3: track 0.00 -> 184.3 mm, vias 0 -> 8
- net IN_L: track 0.00 -> 173.8 mm, vias 0 -> 2
- net MOD1_A: track 0.00 -> 170.9 mm, vias 0 -> 13
- net IN_R: track 0.00 -> 165.5 mm, vias 0 -> 2
- net GATE_A: track 0.00 -> 158.7 mm, vias 0 -> 4
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
Commit message: hw(reva): a 3V3D copper area cools U_REG; power budget in docs
U_REG (AMS1117-3.3 from +12 V) had 14.1 mm2 of B.Cu copper on its tab.
route.py now reserves an L-shaped 227.7 mm2 area at the tab (REG_COPPER,
a 3V3D-owned B.Cu router obstacle) and fills it after routing as a 3V3D
zone, solid to the tab, 0.2 mm clearance. route_check.py gains the gated
step reg_copper (filled 3V3D B.Cu copper on the tab >= 200 mm2) with its
reg_copper and reg_copper_missing sabotages.

The re-route moved a MOD4_A track under the audio sabotage's LED0 track,
which then took that net on save; _beside now lays its track at the first
signed offset clear of foreign copper (audio and lr).

hardware/reva/power_budget.py prints the 3V3D load inventory, dissipation
and Tj; docs/hardware/power-budget.md carries its lines: worst case at
Ta 50 C 104.5 C before, 83.1 C after (TI LM1117 Table 9-2 as the
copper-area proxy, limit 125 C).

Co-Authored-By: HAL 9000 <293417720+bea-ton-k@users.noreply.github.com>
Routing:
- net M6_CH3: track 224.9 -> 25.6 mm, vias 12 -> 0
- net MOD4_A: track 120.8 -> 312.3 mm, vias 9 -> 16
- net IN_L: track 173.8 -> 279.0 mm, vias 2 -> 10
- net M9_CH6: track 138.4 -> 43.2 mm, vias 6 -> 2
- net KEY_REC_A: track 200.6 -> 133.9 mm, vias 10 -> 5
- net LED4: track 94.3 -> 40.5 mm, vias 8 -> 4
- net SR_CLK: track 509.0 -> 556.9 mm, vias 31 -> 23
- net M0_CH5: track 26.5 -> 72.3 mm
- net MUX_S0: track 516.6 -> 553.2 mm, vias 20 -> 21
- net OUT_R: track 127.2 -> 157.3 mm, vias 6 -> 12
- net MUX_EN2: track 56.4 -> 78.5 mm
- net MUX_EN4_SR: track 106.7 -> 87.4 mm
- net LED6: track 95.0 -> 78.1 mm
- net LED0: track 101.9 -> 114.7 mm, vias 2 -> 8
- net 3V3D: track 424.0 -> 436.1 mm, vias 31 -> 28
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- added copper zone on B.Cu, net 3V3D
