File: hardware/reva/kicad/reva.kicad_pcb (KiCad board)
At the start: 4 copper layers, 300.8 x 110 mm, 213 parts, among them J1 IN_L, J10 RESET, J11 MOD4_B, J12 MOD3_B, J13 MOD2_B, J14 MOD1_B, J15 GATE_B, J16 PITCH_B, J17 OUT_L, J18 OUT_R, J2 IN_R, J3 PITCH_A, J4 GATE_A, J5 MOD1_A, J6 MOD2_A, J7 MOD3_A, J8 MOD4_A, J9 CLOCK, SW1 REC_A, SW2 REC_B, SW3 MODBTN, SW4 SHIFTBTN

Commit message: hw(reva): P4-3 footprints carry their schematic links; paths and parity checks
Every footprint gets its KiCad path, full footprint ID, the symbol's fields (hidden, as on the symbol) and DNP; the 40 unconnected pins get KiCad's unconnected-(...) nets (a nameless pin drops the name part). route_check gains paths (against KiCad's own netlist export) and parity (kicad-cli --schematic-parity with a positive control), each with its two sabotages.

Co-Authored-By: HAL 9000 <293417720+bea-ton-k@users.noreply.github.com>
Parts:
- C1, C3, C5, C6, C_SD2: footprint C_0805_2012Metric -> Capacitor_SMD:C_0805_2012Metric
- C10, C11, C12, C13, C14, C15, C16, C17, C18, C19, C2, C20, C21, C22, C4, C7, C8, C9, C_SD1, C_SENSE0, C_SENSE1, C_SENSE2, C_SENSE3: footprint C_0603_1608Metric -> Capacitor_SMD:C_0603_1608Metric
- C_LDO_T: footprint CP_EIA-6032-28_Kemet-C -> Capacitor_Tantalum_SMD:CP_EIA-6032-28_Kemet-C
- D1, D10, D11, D12, D13, D14, D15, D16, D17, D18, D19, D2, D3, D4, D5, D6, D7, D8, D9: footprint LED_D3.0mm -> LED_THT:LED_D3.0mm
- D_N12, D_P12: footprint D_SMA -> Diode_SMD:D_SMA
- J1, J10, J11, J12, J13, J14, J15, J16, J17, J18, J2, J3, J4, J5, J6, J7, J8, J9: footprint Jack_3.5mm_QingPu_WQP-PJ398SM_Vertical_CircularHoles -> Connector_Audio:Jack_3.5mm_QingPu_WQP-PJ398SM_Vertical_CircularHoles
- J_PWR: footprint IDC-Header_2x05_P2.54mm_Vertical -> Connector_IDC:IDC-Header_2x05_P2.54mm_Vertical
- J_SD: footprint SD_Yamaichi_PJS008U-3000-0 -> FireFlow:SD_Yamaichi_PJS008U-3000-0
- R1, R10, R11, R12, R13, R14, R15, R16, R17, R18, R19, R2, R20, R21, R22, R23, R24, R25, R26, R27, R28, R29, R3, R30, R31, R32, R33, R34, R35, R36, R4, R5, R6, R7, R8, R9: footprint R_0603_1608Metric -> Resistor_SMD:R_0603_1608Metric
- RV1, RV10, RV11, RV12, RV13, RV14, RV15, RV16, RV17, RV18, RV19, RV2, RV20, RV21, RV22, RV23, RV24, RV25, RV26, RV27, RV28, RV29, RV3, RV30, RV31, RV32, RV33, RV34, RV35, RV36, RV37, RV38, RV39, RV4, RV40, RV41, RV42, RV43, RV44, RV45, RV46, RV47, RV48, RV49, RV5, RV50, RV51, RV52, RV53, RV54, RV55, RV56, RV57, RV58, RV59, RV6, RV60, RV61, RV62, RV63, RV64, RV65, RV66, RV67, RV68, RV69, RV7, RV70, RV8, RV9: footprint Potentiometer_Alpha_RD901F-40-00D_Single_Vertical -> Potentiometer_THT:Potentiometer_Alpha_RD901F-40-00D_Single_Vertical
- SW1, SW2, SW3, SW4: footprint SW_Push_LP_Button -> Thonk:SW_Push_LP_Button
- TP1, TP10, TP11, TP12, TP13, TP14, TP15, TP2, TP3, TP4, TP5, TP6, TP7, TP8, TP9: footprint TestPoint_Pad_D1.5mm -> TestPoint:TestPoint_Pad_D1.5mm
- U_IN1, U_MUX0, U_MUX1, U_MUX2, U_MUX3, U_MUX4, U_MUX5, U_MUX6, U_MUX7, U_MUX8, U_MUX9, U_SR1, U_SR2, U_SR3, U_SR4, U_SR5: footprint SOIC-16_3.9x9.9mm_P1.27mm -> Package_SO:SOIC-16_3.9x9.9mm_P1.27mm
- U_REG: footprint SOT-223-3_TabPin2 -> Package_TO_SOT_SMD:SOT-223-3_TabPin2
- U_SM: footprint DAISY_PATCH_SM -> Daisy-Boards:DAISY_PATCH_SM
Connections:
- J1 pad TN: (no net) -> unconnected-(J1-PadTN)
- J10 pad TN: (no net) -> unconnected-(J10-PadTN)
- J11 pad TN: (no net) -> unconnected-(J11-PadTN)
- J12 pad TN: (no net) -> unconnected-(J12-PadTN)
- J13 pad TN: (no net) -> unconnected-(J13-PadTN)
- J14 pad TN: (no net) -> unconnected-(J14-PadTN)
- J15 pad TN: (no net) -> unconnected-(J15-PadTN)
- J16 pad TN: (no net) -> unconnected-(J16-PadTN)
- J17 pad TN: (no net) -> unconnected-(J17-PadTN)
- J18 pad TN: (no net) -> unconnected-(J18-PadTN)
- J3 pad TN: (no net) -> unconnected-(J3-PadTN)
- J4 pad TN: (no net) -> unconnected-(J4-PadTN)
- J5 pad TN: (no net) -> unconnected-(J5-PadTN)
- J6 pad TN: (no net) -> unconnected-(J6-PadTN)
- J7 pad TN: (no net) -> unconnected-(J7-PadTN)
- J8 pad TN: (no net) -> unconnected-(J8-PadTN)
- J9 pad TN: (no net) -> unconnected-(J9-PadTN)
- J_PWR pad 7: (no net) -> unconnected-(J_PWR-Pin_7-Pad7)
- J_PWR pad 8: (no net) -> unconnected-(J_PWR-Pin_8-Pad8)
- SW1 pad 3: (no net) -> unconnected-(SW1-C-Pad3)
- SW1 pad 4: (no net) -> unconnected-(SW1-A-Pad4)
- SW1 pad 5: (no net) -> unconnected-(SW1-B-Pad5)
- SW1 pad 6: (no net) -> unconnected-(SW1-C-Pad6)
- SW2 pad 3: (no net) -> unconnected-(SW2-C-Pad3)
- SW2 pad 4: (no net) -> unconnected-(SW2-A-Pad4)
- SW2 pad 5: (no net) -> unconnected-(SW2-B-Pad5)
- SW2 pad 6: (no net) -> unconnected-(SW2-C-Pad6)
- SW3 pad 3: (no net) -> unconnected-(SW3-C-Pad3)
- SW3 pad 4: (no net) -> unconnected-(SW3-A-Pad4)
- SW3 pad 5: (no net) -> unconnected-(SW3-B-Pad5)
- SW3 pad 6: (no net) -> unconnected-(SW3-C-Pad6)
- SW4 pad 3: (no net) -> unconnected-(SW4-C-Pad3)
- SW4 pad 4: (no net) -> unconnected-(SW4-A-Pad4)
- SW4 pad 5: (no net) -> unconnected-(SW4-B-Pad5)
- SW4 pad 6: (no net) -> unconnected-(SW4-C-Pad6)
- U_IN1 pad 7: (no net) -> unconnected-(U_IN1-~{Q7}-Pad7)
- U_SM pad A6: (no net) -> unconnected-(U_SM-+5V-PadA6)
- U_SM pad A8: (no net) -> unconnected-(U_SM-USB_DM-PadA8)
- U_SM pad A9: (no net) -> unconnected-(U_SM-USB_DP-PadA9)
- U_SR5 pad 9: (no net) -> unconnected-(U_SR5-QH'-Pad9)
