File: hardware/reva/kicad/reva.kicad_pcb (KiCad board)
At the start: 4 copper layers, 300.8 x 110 mm, 213 parts, among them J1 IN_L, J10 RESET, J11 MOD4_B, J12 MOD3_B, J13 MOD2_B, J14 MOD1_B, J15 GATE_B, J16 PITCH_B, J17 OUT_L, J18 OUT_R, J2 IN_R, J3 PITCH_A, J4 GATE_A, J5 MOD1_A, J6 MOD2_A, J7 MOD3_A, J8 MOD4_A, J9 CLOCK, SW1 REC_A, SW2 REC_B, SW3 MODBTN, SW4 SHIFTBTN

Commit message: feat(reva): the board follows the 9 mm plate -- routed, KNOWN_PANEL empty but two admitted audio zones
route.py --write is GREEN on the new hole list (73 pots, 15 LEDs, jack
row at 112.75): router 44 rounds, 0 conflicts, 0 failed; drc gated 0;
audio 0 below 10.0 mm and 0 across a zone edge below 3.0 mm; SENSE
factors 1.08 / 1.14 / 1.21 / 1.19; pot_keepout 0; heat copper 351.0 mm2;
no_room 3 hidden, all listed (Bastian).

route_check.KNOWN_PANEL: routed / drc / silk empty; audio keeps the two
jack zones Bastian admitted (renewed 2026-10-07 for the combined lamps):
IN_L/SHIFTBTN_L (J1.T: D1.2, R18.1, R18.2) and MODBTN_L/OUT_R (J18.T:
D15.2). test_route: PAIRS / SONG / CUT_OFF_KEYS empty, ZONE_PAIRS and
JACK_ZONES to the new pairs and members, jack row at y 112.75, the name
rule's fixtures follow (old pairs, SONG and CEIL_L now refused). The
routed_song sabotage finds SONG_A by its panel id and lists the key
itself (the real list is empty), so it still proves the not-a-cut-off
exclusion. P4-2 spec §4.4 carries the amendment.

Co-Authored-By: HAL 9000 <293417720+bea-ton-k@users.noreply.github.com>
Parts:
- removed D16: SONG_B_L, LED_THT:LED_D3.0mm
- removed D17: CEIL_L, LED_THT:LED_D3.0mm
- removed D18: CLR_B_L, LED_THT:LED_D3.0mm
- removed D19: MODBTN_L, LED_THT:LED_D3.0mm
- removed R33, R34, R35, R36: 1k, Resistor_SMD:R_0603_1608Metric
- added RV71: FLUXFB_B, Potentiometer_THT:Potentiometer_Alpha_RD901F-40-00D_Single_Vertical, F.Cu at (255.9, 87.5)
- added RV72: DETUNE_B, Potentiometer_THT:Potentiometer_Alpha_RD901F-40-00D_Single_Vertical, F.Cu at (276.1, 87.5)
- added RV73: ROOT_B, Potentiometer_THT:Potentiometer_Alpha_RD901F-40-00D_Single_Vertical, F.Cu at (296.3, 87.5)
- D10: value TEMPO_L -> REC_B_L
- D11: value REC_B_L -> LVL_B_L
- D12: value LVL_B_L -> FTIME_B_L
- D13: value FLT_B_L -> SONG_B_L
- D14: value SRC_B_L -> GATE_B_L
- D15: value GATE_B_L -> MODBTN_L
- D2: value CLR_A_L -> SONG_A_L
- D3: value SONG_A_L -> GATE_A_L
- D4: value GATE_A_L -> FTIME_A_L
- D5: value SRC_A_L -> LVL_A_L
- D6: value FLT_A_L -> REC_A_L
- D7: value REC_A_L -> CLK_L
- D8: value LVL_A_L -> TEMPO_L
- D9: value SYNC_L -> RST_L
- RV10: value SOURCE_A -> RANGE_A
- RV11: value MOD_A -> ATTACK_A
- RV12: value DENSITY_A -> DECAY_A
- RV13: value TUNE_A -> COLOR_A
- RV14: value DETUNE_A -> TUNE_A
- RV17: value COLOR_A -> ROOT_A
- RV18: value FLUXFB_A -> DETUNE_A
- RV19: value SCALE -> FLUXFB_A
- RV20: value DRIFT -> LINK_A
- RV21: value DECAY_A -> MELODY_A
- RV22: value RES_A -> SCALE
- RV23: value SUB_A -> FILT_A
- RV24: value TEMPO -> DEPTH_A
- RV26: value FILT_A -> RES_A
- RV27: value DEPTH_A -> TEMPO
- RV28: value REV_SIZE -> SUB_A
- RV30: value LINK_A -> PAN_A
- RV31: value PAN_A -> COUPLE
- RV34: value CHOKE -> REV_DIFF
- RV35: value PULL -> CHOKE
- RV36: value COUPLE -> PULL
- RV37: value SHUFFLE -> MELODY_B
- RV38: value SUB_B -> MORPH
- RV41: value MORPH -> SUB_B
- RV42: value REV_DIFF -> REV_SIZE
- RV43: value REV_DECAY -> SHUFFLE
- RV44: value COMP_B -> REV_DECAY
- RV45: value REV_TONE -> DRIFT
- RV46: value REV_MIX_B -> PAN_B
- RV47: value GRIT_B -> REV_TONE
- RV48: value PAN_B -> REV_MOD
- RV49: value MELODY_B -> REV_MIX_B
- RV5: value MELODY_A -> MOD_A
- RV50: value RATE_B -> SONG_B
- RV51: value RES_B -> STEPS_B
- RV52: value DECAY_B -> ENGINE_B
- RV53: value ATTACK_B -> SHAPE_B
- RV54: value SOURCE_B -> MOD_B
- RV55: value FILT_B -> RANGE_B
- RV56: value SONG_B -> SMOOTH_B
- RV57: value STEPS_B -> COLOR_B
- RV58: value ENGINE_B -> RATE_B
- RV59: value RANGE_B -> FILT_B
- RV6: value SMOOTH_A -> SHAPE_A
- RV60: value SMOOTH_B -> SOURCE_B
- RV61: value SHAPE_B -> DENSITY_B
- RV62: value DENSITY_B -> RES_B
- RV63: value MOD_B -> DECAY_B
- RV64: value DETUNE_B -> ATTACK_B
- RV65: value TUNE_B -> COMP_B
- RV66: value FLUX_B -> FLUXRATE_B
- RV67: value LINK_B -> FLUX_B
- RV68: value FLUXRATE_B -> TUNE_B
- RV69: value COLOR_B -> GRIT_B
- RV7: value SHAPE_A -> DENSITY_A
- RV70: value FLUXFB_B -> LINK_B
- RV8: value RANGE_A -> SOURCE_A
- RV9: value ATTACK_A -> SMOOTH_A
- moved C22 114.9 mm to (82.5, 58.9)
- moved U_IN1 114.9 mm to (76.4, 61.3)
- moved C21 112.0 mm to (120.7, 63.5), turned to 90 degrees
- moved TP8 111.9 mm to (123.6, 66.5)
- moved TP9 109.7 mm to (118.3, 61.5)
- moved TP15 108.3 mm to (122.4, 51.5)
- moved TP12 104.5 mm to (120.1, 58.5)
- moved TP10 103.7 mm to (121.6, 55.5)
- moved U_SR5 103.3 mm to (126.7, 61.0), turned to -90 degrees
- moved TP14 102.6 mm to (125.1, 51.5)
- moved D7 101.9 mm to (129.3, 114.0), turned to 90 degrees
- moved RV19 100.7 mm to (53.9, 87.5), turned to -90 degrees
- moved R24 100.5 mm to (127.3, 111.5), turned to 90 degrees
- moved TP11 97.2 mm to (127.8, 55.5)
- moved TP13 96.9 mm to (127.9, 52.5)
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Connections:
- RV10 pad 2: M1_CH3 -> M1_CH1
- RV11 pad 2: M1_CH4 -> M1_CH2
- RV12 pad 2: M1_CH5 -> M1_CH3
- RV19 pad 2: M6_CH0 -> M2_CH6
- RV20 pad 2: M6_CH1 -> M2_CH7
- RV21 pad 2: M6_CH2 -> M6_CH0
- RV22 pad 2: M6_CH3 -> M6_CH1
- RV23 pad 2: M6_CH4 -> M6_CH2
- RV24 pad 2: M6_CH5 -> M6_CH3
- RV25 pad 2: M6_CH6 -> M6_CH4
- RV26 pad 2: M6_CH7 -> M6_CH5
- RV27 pad 2: M7_CH0 -> M6_CH6
- RV28 pad 2: M7_CH1 -> M7_CH0
- RV29 pad 2: M7_CH2 -> M7_CH1
- RV30 pad 2: M7_CH3 -> M7_CH2
- RV31 pad 2: M7_CH4 -> M7_CH3
- RV32 pad 2: M7_CH5 -> M7_CH4
- RV33 pad 2: M7_CH6 -> M7_CH5
- RV34 pad 2: M8_CH0 -> M7_CH6
- RV35 pad 2: M8_CH1 -> M8_CH0
- RV36 pad 2: M8_CH2 -> M8_CH1
- RV37 pad 2: M8_CH3 -> M8_CH2
- RV38 pad 2: M8_CH4 -> M8_CH3
- RV39 pad 2: M8_CH5 -> M8_CH4
- RV40 pad 2: M8_CH6 -> M8_CH5
- RV41 pad 2: M8_CH7 -> M8_CH6
- RV49 pad 2: M3_CH0 -> M9_CH7
- RV50 pad 2: M3_CH1 -> M3_CH0
- RV51 pad 2: M3_CH2 -> M3_CH1
- RV52 pad 2: M3_CH3 -> M3_CH2
- RV53 pad 2: M3_CH4 -> M3_CH3
- RV54 pad 2: M3_CH5 -> M3_CH4
- RV55 pad 2: M3_CH6 -> M3_CH5
- RV56 pad 2: M4_CH0 -> M3_CH6
- RV57 pad 2: M4_CH1 -> M3_CH7
- RV58 pad 2: M4_CH2 -> M4_CH0
- RV59 pad 2: M4_CH3 -> M4_CH1
- RV60 pad 2: M4_CH4 -> M4_CH2
- RV61 pad 2: M4_CH5 -> M4_CH3
- RV62 pad 2: M4_CH6 -> M4_CH4
- RV63 pad 2: M4_CH7 -> M4_CH5
- RV64 pad 2: M5_CH0 -> M4_CH6
- RV65 pad 2: M5_CH1 -> M4_CH7
- RV66 pad 2: M5_CH2 -> M5_CH0
- RV67 pad 2: M5_CH3 -> M5_CH1
- RV68 pad 2: M5_CH4 -> M5_CH2
- RV69 pad 2: M5_CH5 -> M5_CH3
- RV7 pad 2: M1_CH0 -> M0_CH6
- RV70 pad 2: M5_CH6 -> M5_CH4
- RV8 pad 2: M1_CH1 -> M0_CH7
- RV9 pad 2: M1_CH2 -> M1_CH0
- U_MUX0 pad 2: GND -> M0_CH6
- U_MUX0 pad 4: GND -> M0_CH7
- U_MUX1 pad 1: M1_CH4 -> GND
- U_MUX1 pad 2: SM_3V3 -> GND
- U_MUX1 pad 5: M1_CH5 -> SM_3V3
- U_MUX2 pad 2: GND -> M2_CH6
- U_MUX2 pad 4: GND -> M2_CH7
- U_MUX3 pad 4: GND -> M3_CH7
- U_MUX5 pad 4: GND -> M5_CH7
- U_MUX6 pad 4: M6_CH7 -> GND
- U_MUX8 pad 4: M8_CH7 -> GND
- U_MUX9 pad 4: GND -> M9_CH7
- U_SR4 pad 4: LED15 -> unconnected-(U_SR4-QE-Pad4)
- U_SR4 pad 5: LED16 -> unconnected-(U_SR4-QF-Pad5)
- U_SR4 pad 6: LED17 -> unconnected-(U_SR4-QG-Pad6)
- U_SR4 pad 7: LED18 -> unconnected-(U_SR4-QH-Pad7)
Routing:
- net SR_SPARE6: track 8.06 -> 604.4 mm, vias 0 -> 36
- net SR_LATCH: track 228.1 -> 501.9 mm, vias 18 -> 28
- net 3V3D: track 436.1 -> 707.7 mm, vias 28 -> 35
- net SR_CLK: track 556.9 -> 288.1 mm, vias 23 -> 17
- net MOD4_A: track 312.3 -> 71.1 mm, vias 16 -> 5
- net +12V: track 103.5 -> 302.0 mm, vias 7 -> 15
- net IN_L: track 279.0 -> 141.9 mm, vias 10 -> 0
- net KEY_MODBTN: track 117.6 -> 240.7 mm, vias 4 -> 8
- net KEY_REC_B: track 58.2 -> 180.5 mm, vias 2 -> 10
- net SD_D0: track 72.8 -> 192.9 mm, vias 2 -> 8
- net -12V: track 82.3 -> 198.9 mm, vias 4 -> 9
- net SR_CHAIN4: track 24.4 -> 134.3 mm, vias 4 -> 6
- net SENSE_2: track 47.5 -> 130.6 mm, vias 2 -> 3
- net MUX_EN4_SR: track 87.4 -> 157.9 mm, vias 6 -> 12
- net GATE_A: track 158.7 -> 90.6 mm, vias 4 -> 1
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