File: hardware/reva/kicad/mux_sense_0.kicad_sch (KiCad schematic)
At the start: 24 parts

Commit message: feat(reva): 15 LED nets on the 595 chain, four more spare outputs
Spec 2026-10-07 section 5: 15 lamps (LED0..LED14), 73 pots. U_SR4 keeps
LED11..LED14 and gains SR_SPARE8..11, marked no-connect (four more test
points would wrap the chains sheet past the A3 title block). BOMs, review
sheet and the leds / mux sheets regenerated with hardware/reva/build.py.

Co-Authored-By: HAL 9000 <293417720+bea-ton-k@users.noreply.github.com>
Parts:
- added RV19: FLUXFB_A, Potentiometer_THT:Potentiometer_Alpha_RD901F-40-00D_Single_Vertical, symbol Device:R_Potentiometer
- added RV20: LINK_A, Potentiometer_THT:Potentiometer_Alpha_RD901F-40-00D_Single_Vertical, symbol Device:R_Potentiometer
- RV10: value SOURCE_A -> RANGE_A; PanelId SOURCE_A -> RANGE_A
- RV11: value MOD_A -> ATTACK_A; PanelId MOD_A -> ATTACK_A
- RV12: value DENSITY_A -> DECAY_A; PanelId DENSITY_A -> DECAY_A
- RV13: value TUNE_A -> COLOR_A; PanelId TUNE_A -> COLOR_A
- RV14: value DETUNE_A -> TUNE_A; PanelId DETUNE_A -> TUNE_A
- RV17: value COLOR_A -> ROOT_A; PanelId COLOR_A -> ROOT_A
- RV18: value FLUXFB_A -> DETUNE_A; PanelId FLUXFB_A -> DETUNE_A
- RV5: value MELODY_A -> MOD_A; PanelId MELODY_A -> MOD_A
- RV6: value SMOOTH_A -> SHAPE_A; PanelId SMOOTH_A -> SHAPE_A
- RV7: value SHAPE_A -> DENSITY_A; PanelId SHAPE_A -> DENSITY_A
- RV8: value RANGE_A -> SOURCE_A; PanelId RANGE_A -> SOURCE_A
- RV9: value ATTACK_A -> SMOOTH_A; PanelId ATTACK_A -> SMOOTH_A
Connections:
- net GND: now also U_MUX1.1 (A4), U_MUX1.2 (A6), RV19.1, RV20.1; no longer U_MUX0.2 (A6), U_MUX0.4 (A7), U_MUX2.2 (A6), U_MUX2.4 (A7)
- net M1_CH0: now also RV9.2; no longer RV7.2
- net M1_CH1: now also RV10.2; no longer RV8.2
- net M1_CH2: now also RV11.2; no longer RV9.2
- net M1_CH3: now also RV12.2; no longer RV10.2
- net SM_3V3: now also U_MUX1.5 (A5), RV19.3, RV20.3; no longer U_MUX1.2 (A6)
- removed net M1_CH4: RV11.2, U_MUX1.1 (A4)
- removed net M1_CH5: RV12.2, U_MUX1.5 (A5)
- new net M0_CH6: RV7.2, U_MUX0.2 (A6)
- new net M0_CH7: RV8.2, U_MUX0.4 (A7)
- new net M2_CH6: RV19.2, U_MUX2.2 (A6)
- new net M2_CH7: RV20.2, U_MUX2.4 (A7)
