File: hardware/reva/kicad/mux_sense_1.kicad_sch (KiCad schematic)
At the start: 28 parts

Commit message: feat(reva): 15 LED nets on the 595 chain, four more spare outputs
Spec 2026-10-07 section 5: 15 lamps (LED0..LED14), 73 pots. U_SR4 keeps
LED11..LED14 and gains SR_SPARE8..11, marked no-connect (four more test
points would wrap the chains sheet past the A3 title block). BOMs, review
sheet and the leds / mux sheets regenerated with hardware/reva/build.py.

Co-Authored-By: HAL 9000 <293417720+bea-ton-k@users.noreply.github.com>
Parts:
- removed RV49: MELODY_B, Potentiometer_THT:Potentiometer_Alpha_RD901F-40-00D_Single_Vertical, symbol Device:R_Potentiometer
- added RV71: FLUXFB_B, Potentiometer_THT:Potentiometer_Alpha_RD901F-40-00D_Single_Vertical, symbol Device:R_Potentiometer
- added RV72: DETUNE_B, Potentiometer_THT:Potentiometer_Alpha_RD901F-40-00D_Single_Vertical, symbol Device:R_Potentiometer
- added RV73: ROOT_B, Potentiometer_THT:Potentiometer_Alpha_RD901F-40-00D_Single_Vertical, symbol Device:R_Potentiometer
- RV50: value RATE_B -> SONG_B; PanelId RATE_B -> SONG_B
- RV51: value RES_B -> STEPS_B; PanelId RES_B -> STEPS_B
- RV52: value DECAY_B -> ENGINE_B; PanelId DECAY_B -> ENGINE_B
- RV53: value ATTACK_B -> SHAPE_B; PanelId ATTACK_B -> SHAPE_B
- RV54: value SOURCE_B -> MOD_B; PanelId SOURCE_B -> MOD_B
- RV55: value FILT_B -> RANGE_B; PanelId FILT_B -> RANGE_B
- RV56: value SONG_B -> SMOOTH_B; PanelId SONG_B -> SMOOTH_B
- RV57: value STEPS_B -> COLOR_B; PanelId STEPS_B -> COLOR_B
- RV58: value ENGINE_B -> RATE_B; PanelId ENGINE_B -> RATE_B
- RV59: value RANGE_B -> FILT_B; PanelId RANGE_B -> FILT_B
- RV60: value SMOOTH_B -> SOURCE_B; PanelId SMOOTH_B -> SOURCE_B
- RV61: value SHAPE_B -> DENSITY_B; PanelId SHAPE_B -> DENSITY_B
- RV62: value DENSITY_B -> RES_B; PanelId DENSITY_B -> RES_B
- RV63: value MOD_B -> DECAY_B; PanelId MOD_B -> DECAY_B
- RV64: value DETUNE_B -> ATTACK_B; PanelId DETUNE_B -> ATTACK_B
- RV65: value TUNE_B -> COMP_B; PanelId TUNE_B -> COMP_B
- RV66: value FLUX_B -> FLUXRATE_B; PanelId FLUX_B -> FLUXRATE_B
- RV67: value LINK_B -> FLUX_B; PanelId LINK_B -> FLUX_B
- RV68: value FLUXRATE_B -> TUNE_B; PanelId FLUXRATE_B -> TUNE_B
- RV69: value COLOR_B -> GRIT_B; PanelId COLOR_B -> GRIT_B
- RV70: value FLUXFB_B -> LINK_B; PanelId FLUXFB_B -> LINK_B
Connections:
- net GND: now also RV71.1, RV72.1, RV73.1; no longer U_MUX3.4 (A7), U_MUX5.4 (A7)
- net M3_CH0: now also RV50.2
- net M3_CH1: now also RV51.2; no longer RV50.2
- net M3_CH2: now also RV52.2; no longer RV51.2
- net M3_CH3: now also RV53.2; no longer RV52.2
- net M3_CH4: now also RV54.2; no longer RV53.2
- net M3_CH5: now also RV55.2; no longer RV54.2
- net M3_CH6: now also RV56.2; no longer RV55.2
- net M4_CH0: now also RV58.2; no longer RV56.2
- net M4_CH1: now also RV59.2; no longer RV57.2
- net M4_CH2: now also RV60.2; no longer RV58.2
- net M4_CH3: now also RV61.2; no longer RV59.2
- net M4_CH4: now also RV62.2; no longer RV60.2
- net M4_CH5: now also RV63.2; no longer RV61.2
- net M4_CH6: now also RV64.2; no longer RV62.2
- net M4_CH7: now also RV65.2; no longer RV63.2
- net M5_CH0: now also RV66.2; no longer RV64.2
- net M5_CH1: now also RV67.2; no longer RV65.2
- net M5_CH2: now also RV68.2; no longer RV66.2
- net M5_CH3: now also RV69.2; no longer RV67.2
- net M5_CH4: now also RV70.2; no longer RV68.2
- net M5_CH5: now also RV71.2; no longer RV69.2
- net M5_CH6: now also RV72.2; no longer RV70.2
- net SM_3V3: now also RV71.3, RV72.3, RV73.3
- new net M3_CH7: RV57.2, U_MUX3.4 (A7)
- new net M5_CH7: RV73.2, U_MUX5.4 (A7)
Other:
- moved on the sheet: RV50, RV51, RV52, RV53, RV54, RV55, RV56, RV57, RV58, RV59, RV60, RV61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
