File: hardware/reva/kicad/mux_sense_2.kicad_sch (KiCad schematic)
At the start: 19 parts

Commit message: feat(reva): 15 LED nets on the 595 chain, four more spare outputs
Spec 2026-10-07 section 5: 15 lamps (LED0..LED14), 73 pots. U_SR4 keeps
LED11..LED14 and gains SR_SPARE8..11, marked no-connect (four more test
points would wrap the chains sheet past the A3 title block). BOMs, review
sheet and the leds / mux sheets regenerated with hardware/reva/build.py.

Co-Authored-By: HAL 9000 <293417720+bea-ton-k@users.noreply.github.com>
Parts:
- removed RV19: SCALE, Potentiometer_THT:Potentiometer_Alpha_RD901F-40-00D_Single_Vertical, symbol Device:R_Potentiometer
- removed RV20: DRIFT, Potentiometer_THT:Potentiometer_Alpha_RD901F-40-00D_Single_Vertical, symbol Device:R_Potentiometer
- added RV34: REV_DIFF, Potentiometer_THT:Potentiometer_Alpha_RD901F-40-00D_Single_Vertical, symbol Device:R_Potentiometer
- RV21: value DECAY_A -> MELODY_A; PanelId DECAY_A -> MELODY_A
- RV22: value RES_A -> SCALE; PanelId RES_A -> SCALE
- RV23: value SUB_A -> FILT_A; PanelId SUB_A -> FILT_A
- RV24: value TEMPO -> DEPTH_A; PanelId TEMPO -> DEPTH_A
- RV26: value FILT_A -> RES_A; PanelId FILT_A -> RES_A
- RV27: value DEPTH_A -> TEMPO; PanelId DEPTH_A -> TEMPO
- RV28: value REV_SIZE -> SUB_A; PanelId REV_SIZE -> SUB_A
- RV30: value LINK_A -> PAN_A; PanelId LINK_A -> PAN_A
- RV31: value PAN_A -> COUPLE; PanelId PAN_A -> COUPLE
Connections:
- net GND: now also U_MUX6.4 (A7), RV34.1
- net M6_CH0: now also RV21.2
- net M6_CH1: now also RV22.2
- net M6_CH2: now also RV23.2; no longer RV21.2
- net M6_CH3: now also RV24.2; no longer RV22.2
- net M6_CH4: now also RV25.2; no longer RV23.2
- net M6_CH5: now also RV26.2; no longer RV24.2
- net M6_CH6: now also RV27.2; no longer RV25.2
- net M7_CH0: now also RV28.2; no longer RV27.2
- net M7_CH1: now also RV29.2; no longer RV28.2
- net M7_CH2: now also RV30.2; no longer RV29.2
- net M7_CH3: now also RV31.2; no longer RV30.2
- net M7_CH4: now also RV32.2; no longer RV31.2
- net M7_CH5: now also RV33.2; no longer RV32.2
- net M7_CH6: now also RV34.2; no longer RV33.2
- net SM_3V3: now also RV34.3
- removed net M6_CH7: RV26.2, U_MUX6.4 (A7)
Other:
- moved on the sheet: RV21, RV22, RV23, RV24, RV25, RV26, RV27, RV28, RV29, RV30, RV31, RV32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
